File: amplifier.kicad_pcb (KiCad board)
At the start: 2 copper layers, 50 x 35 mm, 24 parts

Commit message: Ручная разводка платы, DRC 0, партномера C1-C3, README и отчёт PDF
Parts:
- moved R1 2.25 mm to (110.0, 86.2)
- moved R2 1.00 mm to (110.0, 90.0)
- moved R3 0.83 mm to (123.5, 88.2), turned to -90 degrees
- turned C1 to -90 degrees
- turned C2 to -90 degrees
- turned C3 to -90 degrees
Routing:
- net +3V3: track 0.00 -> 100.1 mm, vias 0 -> 4
- net -3V3: track 0.00 -> 72.3 mm
- net Net-(DA1-+IN): track 0.00 -> 28.6 mm
- net Net-(DA2--IN): track 0.00 -> 28.4 mm
- net Net-(DA3--IN): track 0.00 -> 27.9 mm
- net Net-(DA2-+IN): track 0.00 -> 23.7 mm
- net /OUT2: track 0.00 -> 17.3 mm
- net /OUT: track 0.00 -> 17.2 mm
- net /OUT1: track 0.00 -> 16.4 mm
- net Net-(DA1--IN): track 0.00 -> 14.9 mm
- net Net-(DA3-+IN): track 0.00 -> 9.83 mm
- net /IN-: track 0.00 -> 4.54 mm
- net /IN+: track 0.00 -> 4.54 mm
- net GND: track 0.00 -> 1.30 mm, vias 0 -> 7
- added copper zone on F.Cu, net GND
