File: amplifier.kicad_sch (KiCad schematic)
At the start: 24 parts

Commit message: Ручная разводка платы, DRC 0, партномера C1-C3, README и отчёт PDF
Parts:
- C1, C3: Manufacturer_Part_Number (none) -> CL21B123KBANNNC
- C2: Manufacturer_Part_Number (none) -> C0805C124K1RACTU
Changed lines of the file:
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@@
 			)
 		)
-		(property "Manufacturer_Part_Number" ""
+		(property "Manufacturer_Part_Number" "CL21B123KBANNNC"
 			(at 71.12 132.08 0)
 			(hide yes)
@@
 			)
 		)
-		(property "Manufacturer_Part_Number" ""
+		(property "Manufacturer_Part_Number" "C0805C124K1RACTU"
 			(at 71.12 116.84 0)
 			(hide yes)
@@
 			)
 		)
-		(property "Manufacturer_Part_Number" ""
+		(property "Manufacturer_Part_Number" "CL21B123KBANNNC"
 			(at 71.12 101.6 0)
 			(hide yes)

Commit message: Основная надпись: БИГЕ.941315.001 Э3, обновлены PDF схемы и отчёт
Other:
- company: (none) -> МГТУ им. Н.Э. Баумана
